Commit message: Added caster wheel. Added macro for left and right wheels. Added material for caster wheel in diff_drive.gazebo

File: catkin_ws/src/diff_drive_description/urdf/diff_drive.xacro (robot description, xacro)
@@ -13,8 +13,9 @@
 <xacro:property name="wheelWidth" value="0.05"/>
 <xacro:property name="wheelRadius" value="0.1"/>
-<xacro:property name="wheelPos" value="0.2"/>
+<xacro:property name="wheelPos" value="${wheelRadius}"/>
 <xacro:property name="wheelMass" value="5"/>
 <xacro:property name="cameraSize" value="0.05"/>
 <xacro:property name="cameraMass" value="0.1"/>
+<!-- base joint -->
 <link name="footprint"/>
 <joint name="base_joint" type="fixed">
@@ -22,4 +23,5 @@
 	<child link="chassis"/>
 </joint>
+<!-- chassis -->
 <link name="chassis">
 <collision>
@@ -42,3 +44,31 @@
 </inertial>
 </link>
+<!-- caster wheel -->
+<joint name="fixed" type="fixed">
+  <parent link="chassis"/>
+  <child link="caster_wheel"/>
+</joint>
+<link name="caster_wheel">
+  <collision>
+    <origin xyz="${casterRadius-chassisLength/2} 0 ${casterRadius-chassisHeight+wheelRadius}" rpy="0 0 0"/>
+    <geometry>
+      <sphere radius="${casterRadius}"/>
+    </geometry>
+  </collision>
+  <visual>
+    <origin xyz="${casterRadius-chassisLength/2} 0 ${casterRadius-chassisHeight+wheelRadius}" rpy="0 0 0"/>
+    <geometry>
+      <sphere radius="${casterRadius}"/>
+    </geometry>
+    <material name="red"/>
+  </visual>
+  <inertial>
+    <origin xyz="${casterRadius-chassisLength/2} 0 ${casterRadius-chassisHeight+wheelRadius}" rpy="0 0 0"/>
+    <mass value="${casterMass}"/>
+    <sphere_inertia m="${casterMass}" r="${casterRadius}"/>
+  </inertial>
+</link>
+<!-- main wheels -->
+<wheel lr="left" tY="1"/>
+<wheel lr="right" tY="-1"/>
 </robot>

File: catkin_ws/src/diff_drive_description/urdf/macros.xacro (robot description, xacro)
@@ -22,3 +22,49 @@
 	/>
 </macro>
+<macro name="wheel" params="lr tY">
+<link name="${lr}_wheel">
+  <collision>
+    <origin xyz="0 0 0" rpy="0 ${PI/2} ${PI/2}" />
+    <geometry>
+      <cylinder length="${wheelWidth}" radius="${wheelRadius}"/>
+    </geometry>
+  </collision>
+  <visual>
+    <origin xyz="0 0 0" rpy="0 ${PI/2} ${PI/2}" />
+    <geometry>
+      <cylinder length="${wheelWidth}" radius="${wheelRadius}"/>
+    </geometry>
+    <material name="black"/>
+  </visual>
+  <inertial>
+    <origin xyz="0 0 0" rpy="0 ${PI/2} ${PI/2}" />
+    <mass value="${wheelMass}"/>
+    <cylinder_inertia m="${wheelMass}" r="${wheelRadius}" h="${wheelWidth}"/>
+  </inertial>
+</link>
+<gazebo reference="${lr}_wheel">
+  <mu1 value="1.0"/>
+  <mu2 value="1.0"/>
+  <kp  value="10000000.0" />
+  <kd  value="1.0" />
+  <fdir1 value="1 0 0"/>
+  <material>Gazebo/Black</material>
+</gazebo>
+<joint name="${lr}_wheel_hinge" type="continuous">
+  <parent link="chassis"/>
+  <child link="${lr}_wheel"/>
+<origin xyz="${-wheelPos+chassisLength/2} ${tY*wheelWidth/2+tY*chassisWidth/2} ${wheelRadius}" rpy="0 0 0" />
+  <axis xyz="0 1 0" rpy="0 0 0" />
+  <limit effort="100" velocity="100"/>
+  <joint_properties damping="0.0" friction="0.0"/>
+</joint>
+<transmission name="${lr}_trans">
+  <type>transmission_interface/SimpleTransmission</type>
+  <joint name="${lr}_wheel_hinge"/>
+  <actuator name="${lr}Motor">
+    <hardwareInterface>EffortJointInterface</hardwareInterface>
+    <mechanicalReduction>10</mechanicalReduction>
+  </actuator>
+</transmission>
+</macro>
 </robot>

Commit message: Added rviz launch file, modification of display.launch from urdf_tutorial. Changed base_joint to base_link in diff_drive.xacro for proper RVIZ handling.

File: catkin_ws/src/diff_drive_description/urdf/diff_drive.xacro (robot description, xacro)
@@ -18,7 +18,7 @@
 <xacro:property name="cameraMass" value="0.1"/>
 <!-- base joint -->
-<link name="footprint"/>
+<link name="base_link"/>
 <joint name="base_joint" type="fixed">
-	<parent link="footprint"/>
+	<parent link="base_link"/>
 	<child link="chassis"/>
 </joint>

Commit message: Added laser sensor link and joint to xacro file.

File: catkin_ws/src/diff_drive_description/urdf/diff_drive.xacro (robot description, xacro)
@@ -15,6 +15,7 @@
 <xacro:property name="wheelPos" value="${wheelRadius}"/>
 <xacro:property name="wheelMass" value="5"/>
-<xacro:property name="cameraSize" value="0.05"/>
-<xacro:property name="cameraMass" value="0.1"/>
+<xacro:property name="laserHeight" value="0.1"/>
+<xacro:property name="laserRadius" value="0.05"/>
+<xacro:property name="laserMass" value="0.1"/>
 <!-- base joint -->
 <link name="base_link"/>
@@ -72,3 +73,30 @@
 <wheel lr="left" tY="1"/>
 <wheel lr="right" tY="-1"/>
+<!-- laser sensor -->
+<link name="hokuyo_link">
+	<collision>
+		<origin xyz="0 0 0" rpy="0 0 0"/>
+		<geometry>
+			<cylinder radius="${laserRadius}" length="${laserHeight}"/>
+		</geometry>
+	</collision>
+	<visual>
+		<origin xyz="0 0 0" rpy="0 0 0"/>
+		<geometry>
+			<cylinder radius="${laserRadius}" length="${laserHeight}"/>
+		</geometry>
+		<material name="white"/>
+	</visual>
+	<inertial>
+		<origin xyz="0 0 0" rpy="0 0 0"/>
+		<mass value="${laserMass}"/>
+		<cylinder_inertia m="${laserMass}" r="${laserRadius}" h="${laserHeight}"/>
+	</inertial>
+</link>
+<joint name="hokuyo_joint" type="fixed">
+	<axis xyz="0 1 0"/>
+	<origin xyz="${casterRadius-chassisLength/2} 0 ${chassisHeight+wheelRadius}" rpy="0 0 0"/>
+	<parent link="base_link"/>
+	<child link="hokuyo_link"/>
+</joint>
 </robot>

Commit message: Added joints to each link, added offsets to each joint, removed visual/collision/inertial origin offsets where unnecessary.

File: catkin_ws/src/diff_drive_description/urdf/diff_drive.xacro (robot description, xacro)
@@ -19,11 +19,11 @@
 <xacro:property name="laserMass" value="0.1"/>
 <!-- base joint -->
-<link name="base_link"/>
+<!--<link name="base_link"/>
 <joint name="base_joint" type="fixed">
 	<parent link="base_link"/>
 	<child link="chassis"/>
-</joint>
+</joint>-->
 <!-- chassis -->
-<link name="chassis">
+<link name="base_link">
 <collision>
 	<origin xyz="0 0 ${wheelRadius}" rpy="0 0 0"/>
@@ -46,11 +46,13 @@
 </link>
 <!-- caster wheel -->
-<joint name="fixed" type="fixed">
-  <parent link="chassis"/>
-  <child link="caster_wheel"/>
+<joint name="front_caster_joint" type="continuous">
+	<axis xyz="0 0 1"/>
+	<origin xyz="${casterRadius-chassisLength/2} 0 ${casterRadius-chassisHeight+wheelRadius}" rpy="0 0 0"/>
+  <parent link="base_link"/>
+  <child link="front_caster"/>
 </joint>
-<link name="caster_wheel">
+<link name="front_caster">
   <collision>
-    <origin xyz="${casterRadius-chassisLength/2} 0 ${casterRadius-chassisHeight+wheelRadius}" rpy="0 0 0"/>
+    <origin xyz="0 0 0" rpy="0 0 0"/>
     <geometry>
       <sphere radius="${casterRadius}"/>
@@ -58,5 +60,5 @@
   </collision>
   <visual>
-    <origin xyz="${casterRadius-chassisLength/2} 0 ${casterRadius-chassisHeight+wheelRadius}" rpy="0 0 0"/>
+    <origin xyz="0 0 0" rpy="0 0 0"/>
     <geometry>
       <sphere radius="${casterRadius}"/>
@@ -65,5 +67,5 @@
   </visual>
   <inertial>
-    <origin xyz="${casterRadius-chassisLength/2} 0 ${casterRadius-chassisHeight+wheelRadius}" rpy="0 0 0"/>
+    <origin xyz="0 0 0" rpy="0 0 0"/>
     <mass value="${casterMass}"/>
     <sphere_inertia m="${casterMass}" r="${casterRadius}"/>

File: catkin_ws/src/diff_drive_description/urdf/macros.xacro (robot description, xacro)
@@ -52,5 +52,5 @@
 </gazebo>
 <joint name="${lr}_wheel_hinge" type="continuous">
-  <parent link="chassis"/>
+  <parent link="base_link"/>
   <child link="${lr}_wheel"/>
 <origin xyz="${-wheelPos+chassisLength/2} ${tY*wheelWidth/2+tY*chassisWidth/2} ${wheelRadius}" rpy="0 0 0" />

Commit message: Revert "Added joints to each link, added offsets to each joint, removed visual/collision/inertial origin offsets where unnecessary."
This reverts commit a05f36f9c8ee1ee1c28bb0e24d7401d7f6ffbc6a.

File: catkin_ws/src/diff_drive_description/urdf/diff_drive.xacro (robot description, xacro)
@@ -19,11 +19,11 @@
 <xacro:property name="laserMass" value="0.1"/>
 <!-- base joint -->
-<!--<link name="base_link"/>
+<link name="base_link"/>
 <joint name="base_joint" type="fixed">
 	<parent link="base_link"/>
 	<child link="chassis"/>
-</joint>-->
+</joint>
 <!-- chassis -->
-<link name="base_link">
+<link name="chassis">
 <collision>
 	<origin xyz="0 0 ${wheelRadius}" rpy="0 0 0"/>
@@ -46,13 +46,11 @@
 </link>
 <!-- caster wheel -->
-<joint name="front_caster_joint" type="continuous">
-	<axis xyz="0 0 1"/>
-	<origin xyz="${casterRadius-chassisLength/2} 0 ${casterRadius-chassisHeight+wheelRadius}" rpy="0 0 0"/>
-  <parent link="base_link"/>
-  <child link="front_caster"/>
+<joint name="fixed" type="fixed">
+  <parent link="chassis"/>
+  <child link="caster_wheel"/>
 </joint>
-<link name="front_caster">
+<link name="caster_wheel">
   <collision>
-    <origin xyz="0 0 0" rpy="0 0 0"/>
+    <origin xyz="${casterRadius-chassisLength/2} 0 ${casterRadius-chassisHeight+wheelRadius}" rpy="0 0 0"/>
     <geometry>
       <sphere radius="${casterRadius}"/>
@@ -60,5 +58,5 @@
   </collision>
   <visual>
-    <origin xyz="0 0 0" rpy="0 0 0"/>
+    <origin xyz="${casterRadius-chassisLength/2} 0 ${casterRadius-chassisHeight+wheelRadius}" rpy="0 0 0"/>
     <geometry>
       <sphere radius="${casterRadius}"/>
@@ -67,5 +65,5 @@
   </visual>
   <inertial>
-    <origin xyz="0 0 0" rpy="0 0 0"/>
+    <origin xyz="${casterRadius-chassisLength/2} 0 ${casterRadius-chassisHeight+wheelRadius}" rpy="0 0 0"/>
     <mass value="${casterMass}"/>
     <sphere_inertia m="${casterMass}" r="${casterRadius}"/>

File: catkin_ws/src/diff_drive_description/urdf/macros.xacro (robot description, xacro)
@@ -52,5 +52,5 @@
 </gazebo>
 <joint name="${lr}_wheel_hinge" type="continuous">
-  <parent link="base_link"/>
+  <parent link="chassis"/>
   <child link="${lr}_wheel"/>
 <origin xyz="${-wheelPos+chassisLength/2} ${tY*wheelWidth/2+tY*chassisWidth/2} ${wheelRadius}" rpy="0 0 0" />

Commit message: Added laser scanner and callback, incorporated range reading into avoid_obstacles.cpp, restored driving functionality.

File: catkin_ws/src/diff_drive_description/urdf/diff_drive.xacro (robot description, xacro)
@@ -96,5 +96,5 @@
 <joint name="hokuyo_joint" type="fixed">
 	<axis xyz="0 1 0"/>
-	<origin xyz="${casterRadius-chassisLength/2} 0 ${chassisHeight+wheelRadius}" rpy="0 0 0"/>
+	<origin xyz="${casterRadius-chassisLength/2} 0 ${chassisHeight+wheelRadius}" rpy="0 0 ${PI}"/>
 	<parent link="base_link"/>
 	<child link="hokuyo_link"/>

Commit message: Added avoid obstacles logic to state machine. Added vector heading and driving logic to avoid obstacles. Changed urdf so lidar points toward x direction.

File: catkin_ws/src/diff_drive_description/urdf/diff_drive.xacro (robot description, xacro)
@@ -52,5 +52,5 @@
 <link name="caster_wheel">
   <collision>
-    <origin xyz="${casterRadius-chassisLength/2} 0 ${casterRadius-chassisHeight+wheelRadius}" rpy="0 0 0"/>
+    <origin xyz="${chassisLength/2-casterRadius} 0 ${casterRadius-chassisHeight+wheelRadius}" rpy="0 0 0"/>
     <geometry>
       <sphere radius="${casterRadius}"/>
@@ -58,5 +58,5 @@
   </collision>
   <visual>
-    <origin xyz="${casterRadius-chassisLength/2} 0 ${casterRadius-chassisHeight+wheelRadius}" rpy="0 0 0"/>
+    <origin xyz="${chassisLength/2-casterRadius} 0 ${casterRadius-chassisHeight+wheelRadius}" rpy="0 0 0"/>
     <geometry>
       <sphere radius="${casterRadius}"/>
@@ -65,5 +65,5 @@
   </visual>
   <inertial>
-    <origin xyz="${casterRadius-chassisLength/2} 0 ${casterRadius-chassisHeight+wheelRadius}" rpy="0 0 0"/>
+    <origin xyz="${chassisLength/2-casterRadius} 0 ${casterRadius-chassisHeight+wheelRadius}" rpy="0 0 0"/>
     <mass value="${casterMass}"/>
     <sphere_inertia m="${casterMass}" r="${casterRadius}"/>
@@ -96,5 +96,5 @@
 <joint name="hokuyo_joint" type="fixed">
 	<axis xyz="0 1 0"/>
-	<origin xyz="${casterRadius-chassisLength/2} 0 ${chassisHeight+wheelRadius}" rpy="0 0 ${PI}"/>
+	<origin xyz="${chassisLength/2-casterRadius} 0 ${chassisHeight+wheelRadius}" rpy="0 0 0"/>
 	<parent link="base_link"/>
 	<child link="hokuyo_link"/>

File: catkin_ws/src/diff_drive_description/urdf/macros.xacro (robot description, xacro)
@@ -54,5 +54,5 @@
   <parent link="chassis"/>
   <child link="${lr}_wheel"/>
-<origin xyz="${-wheelPos+chassisLength/2} ${tY*wheelWidth/2+tY*chassisWidth/2} ${wheelRadius}" rpy="0 0 0" />
+<origin xyz="${wheelPos-chassisLength/2} ${tY*wheelWidth/2+tY*chassisWidth/2} ${wheelRadius}" rpy="0 0 0" />
   <axis xyz="0 1 0" rpy="0 0 0" />
   <limit effort="100" velocity="100"/>
